File: olkbd_ble.sch (KiCad schematic (older format))
At the start: 121 parts, among them K1 KEYSW, K10 KEYSW, K11 KEYSW, K12 KEYSW, K13 KEYSW, K14 KEYSW, K15 KEYSW, K16 KEYSW, K17 KEYSW, K18 KEYSW, K19 KEYSW, K2 KEYSW, K20 KEYSW, K21 KEYSW, K22 KEYSW, K23 KEYSW, K24 KEYSW, K25 KEYSW, K26 KEYSW, K27 KEYSW, K28 KEYSW, K29 KEYSW, K3 KEYSW, K30 KEYSW, K31 KEYSW, K32 KEYSW, K33 KEYSW, K34 KEYSW, K35 KEYSW, K36 KEYSW, K37 KEYSW, K38 KEYSW, K39 KEYSW, K4 KEYSW, K40 KEYSW, K41 KEYSW, K42 KEYSW, K43 KEYSW, K44 KEYSW, K45 KEYSW, K46 KEYSW, K47 KEYSW, K48 KEYSW, K49 KEYSW, K5 KEYSW, K50 KEYSW, K51 KEYSW, K52 KEYSW, K53 KEYSW, K54 KEYSW, K55 KEYSW, K56 KEYSW, K57 KEYSW, K58 KEYSW, K59 KEYSW, K6 KEYSW, K60 KEYSW, K7 KEYSW, K8 KEYSW, K9 KEYSW, U1 Lolin32

Commit message: Adding LEDs.
Parts:
- added L1, L10, L11, L12, L13, L14, L15, L16, L17, L18, L19, L2, L20, L21, L22, L23, L24, L25, L26, L27, L28, L29, L3, L30, L31, L32, L33, L34, L35, L36, L37, L38, L39, L4, L40, L41, L42, L43, L44, L45, L46, L47, L48, L49, L5, L50, L51, L52, L53, L54, L55, L56, L57, L58, L59, L6, L60, L7, L8, L9: LED_sk2812_SM, SofleRGB:SK6812MINI_and_cherry, symbol SofleKeyboard:LED_sk2812_SM
- added U2: 0.91_oled_128x32, footprints:0.91_oled_128x32, symbol symbols:0.91_oled_128x32
- D1, D10, D11, D12, D13, D14, D15, D16, D17, D18, D19, D2, D20, D21, D22, D23, D24, D25, D26, D27, D28, D29, D3, D30, D31, D32, D33, D34, D35, D36, D37, D38, D39, D4, D40, D41, D42, D43, D44, D45, D46, D47, D48, D49, D5, D50, D51, D52, D53, D54, D55, D56, D57, D58, D59, D6, D60, D7, D8, D9: footprint keyboard_parts:D_SOD123 -> keyboard_parts:D_SOD123_hand
Connections:
- net GND: now also U1.17 (GND), U1.23 (GND), U1.24 (GND), U1.34 (GND), L1.2 (VSS), L10.2 (VSS), L11.2 (VSS), L12.2 (VSS), L13.2 (VSS), L14.2 (VSS), L15.2 (VSS), L16.2 (VSS), L17.2 (VSS), L18.2 (VSS), L19.2 (VSS), L2.2 (VSS), L20.2 (VSS), L21.2 (VSS), L22.2 (VSS), L23.2 (VSS), L24.2 (VSS), L25.2 (VSS), L26.2 (VSS), L27.2 (VSS), L28.2 (VSS), L29.2 (VSS), L3.2 (VSS), L30.2 (VSS), L31.2 (VSS), L32.2 (VSS), L33.2 (VSS), L34.2 (VSS), L35.2 (VSS), L36.2 (VSS), L37.2 (VSS), L38.2 (VSS), L39.2 (VSS), L4.2 (VSS), L40.2 (VSS), L41.2 (VSS), L42.2 (VSS), L43.2 (VSS), L44.2 (VSS), L45.2 (VSS), L46.2 (VSS), L47.2 (VSS), L48.2 (VSS), L49.2 (VSS), L5.2 (VSS), L50.2 (VSS), L51.2 (VSS), L52.2 (VSS), L53.2 (VSS), L54.2 (VSS), L55.2 (VSS), L56.2 (VSS), L57.2 (VSS), L58.2 (VSS), L59.2 (VSS), L6.2 (VSS), L60.2 (VSS), L7.2 (VSS), L8.2 (VSS), L9.2 (VSS), U2.1 (GND)
- net VCC: now reaches U1.1 (3V)
- net VCC: now also U1.20 (3V), U1.29 (3V), L1.4 (VDD), L10.4 (VDD), L11.4 (VDD), L12.4 (VDD), L13.4 (VDD), L14.4 (VDD), L15.4 (VDD), L16.4 (VDD), L17.4 (VDD), L18.4 (VDD), L19.4 (VDD), L2.4 (VDD), L20.4 (VDD), L21.4 (VDD), L22.4 (VDD), L23.4 (VDD), L24.4 (VDD), L25.4 (VDD), L26.4 (VDD), L27.4 (VDD), L28.4 (VDD), L29.4 (VDD), L3.4 (VDD), L30.4 (VDD), L31.4 (VDD), L32.4 (VDD), L33.4 (VDD), L34.4 (VDD), L35.4 (VDD), L36.4 (VDD), L37.4 (VDD), L38.4 (VDD), L39.4 (VDD), L4.4 (VDD), L40.4 (VDD), L41.4 (VDD), L42.4 (VDD), L43.4 (VDD), L44.4 (VDD), L45.4 (VDD), L46.4 (VDD), L47.4 (VDD), L48.4 (VDD), L49.4 (VDD), L5.4 (VDD), L50.4 (VDD), L51.4 (VDD), L52.4 (VDD), L53.4 (VDD), L54.4 (VDD), L55.4 (VDD), L56.4 (VDD), L57.4 (VDD), L58.4 (VDD), L59.4 (VDD), L6.4 (VDD), L60.4 (VDD), L7.4 (VDD), L8.4 (VDD), L9.4 (VDD), U2.2 (VCC)
- net at U1.21 (SCL/22): now also U2.3 (SCL)
- net at U1.22 (SDA/21): now also U2.4 (SDA)
- net LED: now reaches U1.28 (SS/5/LED)
- net LED: now also L1.3 (DIN)
- new net: L5.1 (DOUT), L6.3 (DIN)
- new net: L4.1 (DOUT), L5.3 (DIN)
- new net: L3.1 (DOUT), L4.3 (DIN)
- new net: L2.1 (DOUT), L3.3 (DIN)
- new net: L1.1 (DOUT), L2.3 (DIN)
- new net: L10.1 (DOUT), L11.3 (DIN)
- new net: L10.3 (DIN), L9.1 (DOUT)
- new net: L8.1 (DOUT), L9.3 (DIN)
- new net: L7.1 (DOUT), L8.3 (DIN)
- new net: L6.1 (DOUT), L7.3 (DIN)
- new net: L15.1 (DOUT), L16.3 (DIN)
- new net: L14.1 (DOUT), L15.3 (DIN)
- new net: L13.1 (DOUT), L14.3 (DIN)
- new net: L12.1 (DOUT), L13.3 (DIN)
- new net: L11.1 (DOUT), L12.3 (DIN)
- new net: L20.1 (DOUT), L21.3 (DIN)
- new net: L19.1 (DOUT), L20.3 (DIN)
- new net: L18.1 (DOUT), L19.3 (DIN)
- new net: L17.1 (DOUT), L18.3 (DIN)
- new net: L16.1 (DOUT), L17.3 (DIN)
- new net: L25.1 (DOUT), L26.3 (DIN)
- new net: L24.1 (DOUT), L25.3 (DIN)
- new net: L23.1 (DOUT), L24.3 (DIN)
- new net: L22.1 (DOUT), L23.3 (DIN)
- new net: L21.1 (DOUT), L22.3 (DIN)
- new net: L30.1 (DOUT), L31.3 (DIN)
- new net: L29.1 (DOUT), L30.3 (DIN)
- new net: L28.1 (DOUT), L29.3 (DIN)
- new net: L27.1 (DOUT), L28.3 (DIN)
- new net: L26.1 (DOUT), L27.3 (DIN)
- new net: L35.1 (DOUT), L36.3 (DIN)
- new net: L34.1 (DOUT), L35.3 (DIN)
- new net: L33.1 (DOUT), L34.3 (DIN)
- new net: L32.1 (DOUT), L33.3 (DIN)
- new net: L31.1 (DOUT), L32.3 (DIN)
- new net: L40.1 (DOUT), L41.3 (DIN)
- new net: L39.1 (DOUT), L40.3 (DIN)
- new net: L38.1 (DOUT), L39.3 (DIN)
- new net: L37.1 (DOUT), L38.3 (DIN)
- new net: L36.1 (DOUT), L37.3 (DIN)
- new net: L45.1 (DOUT), L46.3 (DIN)
- new net: L44.1 (DOUT), L45.3 (DIN)
- new net: L43.1 (DOUT), L44.3 (DIN)
- new net: L42.1 (DOUT), L43.3 (DIN)
- new net: L41.1 (DOUT), L42.3 (DIN)
- new net: L50.1 (DOUT), L51.3 (DIN)
- new net: L49.1 (DOUT), L50.3 (DIN)
- new net: L48.1 (DOUT), L49.3 (DIN)
- new net: L47.1 (DOUT), L48.3 (DIN)
- new net: L46.1 (DOUT), L47.3 (DIN)
- new net: L55.1 (DOUT), L56.3 (DIN)
- new net: L54.1 (DOUT), L55.3 (DIN)
- new net: L53.1 (DOUT), L54.3 (DIN)
- new net: L52.1 (DOUT), L53.3 (DIN)
- new net: L51.1 (DOUT), L52.3 (DIN)
- new net: L59.1 (DOUT), L60.3 (DIN)
- new net: L58.1 (DOUT), L59.3 (DIN)
- new net: L57.1 (DOUT), L58.3 (DIN)
- new net: L56.1 (DOUT), L57.3 (DIN)
Other:
- moved on the sheet: D1, D10, D11, D12, D13, D14, D15, D16, D17, D18, D19, D2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
