File: olkbd_ble.kicad_pcb (KiCad board)
At the start: 2 copper layers, 261 x 97 mm, 121 parts, among them K1 KEYSW, K10 KEYSW, K11 KEYSW, K12 KEYSW, K13 KEYSW, K14 KEYSW, K15 KEYSW, K16 KEYSW, K17 KEYSW, K18 KEYSW, K19 KEYSW, K2 KEYSW, K20 KEYSW, K21 KEYSW, K22 KEYSW, K23 KEYSW, K24 KEYSW, K25 KEYSW, K26 KEYSW, K27 KEYSW, K28 KEYSW, K29 KEYSW, K3 KEYSW, K30 KEYSW, K31 KEYSW, K32 KEYSW, K33 KEYSW, K34 KEYSW, K35 KEYSW, K36 KEYSW, K37 KEYSW, K38 KEYSW, K39 KEYSW, K4 KEYSW, K40 KEYSW, K41 KEYSW, K42 KEYSW, K43 KEYSW, K44 KEYSW, K45 KEYSW, K46 KEYSW, K47 KEYSW, K48 KEYSW, K49 KEYSW, K5 KEYSW, K50 KEYSW, K51 KEYSW, K52 KEYSW, K53 KEYSW, K54 KEYSW, K55 KEYSW, K56 KEYSW, K57 KEYSW, K58 KEYSW, K59 KEYSW, K6 KEYSW, K60 KEYSW, K7 KEYSW, K8 KEYSW, K9 KEYSW, U1 Lolin32

Commit message: Finalized. Need blings.
Routing:
- net ROW3: track 0.00 -> 382.3 mm
- net ROW0: track 0.00 -> 375.2 mm
- net COL11: track 0.00 -> 343.1 mm
- net COL10: track 0.00 -> 335.0 mm, vias 0 -> 1
- net COL9: track 0.00 -> 323.9 mm, vias 0 -> 1
- net ROW2: track 0.00 -> 284.0 mm, vias 0 -> 5
- net ROW1: track 0.00 -> 280.9 mm, vias 0 -> 4
- net ROW4: track 0.00 -> 277.9 mm
- net COL8: track 0.00 -> 275.3 mm, vias 0 -> 1
- net COL7: track 0.00 -> 270.9 mm, vias 0 -> 1
- net COL6: track 0.00 -> 216.2 mm, vias 0 -> 2
- net COL5: track 0.00 -> 198.1 mm, vias 0 -> 2
- net COL0: track 0.00 -> 187.4 mm, vias 0 -> 1
- net COL3: track 0.00 -> 183.1 mm, vias 0 -> 1
- net COL4: track 0.00 -> 175.6 mm, vias 0 -> 2
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Other:
- board size 261 x 97 mm -> 259.6 x 309.6 mm

Commit message: v1.0 ready for oshpark.
Parts:
- added G***: LOGO, testboard:logo, F.Cu at (223.8, 271.5)
- added G***: LOGO, testboard:logo, F.Cu at (223.8, 328.6)
- added G***: LOGO, testboard:logo, F.Cu at (281.0, 302.4)
- added G***: LOGO, testboard:logo, F.Cu at (166.7, 302.4)
Routing:
- net GND: vias 0 -> 22
- net (no net): vias 63 -> 41
- added copper zone on B.Cu, net GND
- added copper zone on F.Cu, net GND
Other:
- board size 259.6 x 309.6 mm -> 259.6 x 290.5 mm
- board text added: "CatiONE OLKB v1.0"
- board text added: "Dung Phan 2021"
- board text added: "Powered by MK32 https://github.com/Galzai/MK32"

Commit message: Panelizing in kicad.
Parts:
- added mouse-bite-2mm-slot: VAL**, Panelization:mouse-bite-2mm-slot, F.Cu at (300.0, 251.0)
- added mouse-bite-2mm-slot: VAL**, Panelization:mouse-bite-2mm-slot, F.Cu at (224.0, 251.0)
- added mouse-bite-2mm-slot: VAL**, Panelization:mouse-bite-2mm-slot, F.Cu at (147.0, 251.0)
- added mouse-bite-2mm-slot: VAL**, Panelization:mouse-bite-2mm-slot, F.Cu at (147.0, 153.8)
- added mouse-bite-2mm-slot: VAL**, Panelization:mouse-bite-2mm-slot, F.Cu at (224.0, 153.8)
- added mouse-bite-2mm-slot: VAL**, Panelization:mouse-bite-2mm-slot, F.Cu at (300.0, 153.8)
- moved K58 2.42 mm to (328.5, 202.4)
- moved K13 2.42 mm to (157.0, 202.4)
- moved K28 2.42 mm to (214.2, 202.4)
- moved K38 2.42 mm to (252.3, 202.4)
- moved K3 2.42 mm to (118.9, 202.4)
- moved K18 2.42 mm to (176.1, 202.4)
- moved K23 2.42 mm to (195.1, 202.4)
- moved K33 2.42 mm to (233.2, 202.4)
- moved K43 2.42 mm to (271.3, 202.4)
- moved K48 2.42 mm to (290.4, 202.4)
- moved K53 2.42 mm to (309.4, 202.4)
- moved K8 2.42 mm to (138.0, 202.4)
- moved K56 2.42 mm to (328.5, 164.3)
- moved K57 2.42 mm to (328.5, 183.3)
- moved K59 2.42 mm to (328.5, 221.4)
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Connections:
- D1 pad 1: ROW0 -> (no net)
- D1 pad 2: Net-(D1-Pad2) -> (no net)
- D10 pad 1: ROW4 -> (no net)
- D10 pad 2: Net-(D10-Pad2) -> (no net)
- D11 pad 1: ROW0 -> (no net)
- D11 pad 2: Net-(D11-Pad2) -> (no net)
- D12 pad 1: ROW1 -> (no net)
- D12 pad 2: Net-(D12-Pad2) -> (no net)
- D13 pad 1: ROW2 -> (no net)
- D13 pad 2: Net-(D13-Pad2) -> (no net)
- D14 pad 1: ROW3 -> (no net)
- D14 pad 2: Net-(D14-Pad2) -> (no net)
- D15 pad 1: ROW4 -> (no net)
- D15 pad 2: Net-(D15-Pad2) -> (no net)
- D16 pad 1: ROW0 -> (no net)
- D16 pad 2: Net-(D16-Pad2) -> (no net)
- D17 pad 1: ROW1 -> (no net)
- D17 pad 2: Net-(D17-Pad2) -> (no net)
- D18 pad 1: ROW2 -> (no net)
- D18 pad 2: Net-(D18-Pad2) -> (no net)
- D19 pad 1: ROW3 -> (no net)
- D19 pad 2: Net-(D19-Pad2) -> (no net)
- D2 pad 1: ROW1 -> (no net)
- D2 pad 2: Net-(D2-Pad2) -> (no net)
- D20 pad 1: ROW4 -> (no net)
- D20 pad 2: Net-(D20-Pad2) -> (no net)
- D21 pad 1: ROW0 -> (no net)
- D21 pad 2: Net-(D21-Pad2) -> (no net)
- D22 pad 1: ROW1 -> (no net)
- D22 pad 2: Net-(D22-Pad2) -> (no net)
- D23 pad 1: ROW2 -> (no net)
- D23 pad 2: Net-(D23-Pad2) -> (no net)
- D24 pad 1: ROW3 -> (no net)
- D24 pad 2: Net-(D24-Pad2) -> (no net)
- D25 pad 1: ROW4 -> (no net)
- D25 pad 2: Net-(D25-Pad2) -> (no net)
- D26 pad 1: ROW0 -> (no net)
- D26 pad 2: Net-(D26-Pad2) -> (no net)
- D27 pad 1: ROW1 -> (no net)
- D27 pad 2: Net-(D27-Pad2) -> (no net)
- D28 pad 1: ROW2 -> (no net)
- D28 pad 2: Net-(D28-Pad2) -> (no net)
- D29 pad 1: ROW3 -> (no net)
- D29 pad 2: Net-(D29-Pad2) -> (no net)
- D3 pad 1: ROW2 -> (no net)
- D3 pad 2: Net-(D3-Pad2) -> (no net)
- D30 pad 1: ROW4 -> (no net)
- D30 pad 2: Net-(D30-Pad2) -> (no net)
- D31 pad 1: ROW0 -> (no net)
- D31 pad 2: Net-(D31-Pad2) -> (no net)
- D32 pad 1: ROW1 -> (no net)
- D32 pad 2: Net-(D32-Pad2) -> (no net)
- D33 pad 1: ROW2 -> (no net)
- D33 pad 2: Net-(D33-Pad2) -> (no net)
- D34 pad 1: ROW3 -> (no net)
- D34 pad 2: Net-(D34-Pad2) -> (no net)
- D35 pad 1: ROW4 -> (no net)
- D35 pad 2: Net-(D35-Pad2) -> (no net)
- D36 pad 1: ROW0 -> (no net)
- D36 pad 2: Net-(D36-Pad2) -> (no net)
- D37 pad 1: ROW1 -> (no net)
- D37 pad 2: Net-(D37-Pad2) -> (no net)
- D38 pad 1: ROW2 -> (no net)
- D38 pad 2: Net-(D38-Pad2) -> (no net)
- D39 pad 1: ROW3 -> (no net)
- D39 pad 2: Net-(D39-Pad2) -> (no net)
- D4 pad 1: ROW3 -> (no net)
- D4 pad 2: Net-(D4-Pad2) -> (no net)
- D40 pad 1: ROW4 -> (no net)
- D40 pad 2: Net-(D40-Pad2) -> (no net)
- D41 pad 1: ROW0 -> (no net)
- D41 pad 2: Net-(D41-Pad2) -> (no net)
- D42 pad 1: ROW1 -> (no net)
- D42 pad 2: Net-(D42-Pad2) -> (no net)
- D43 pad 1: ROW2 -> (no net)
- D43 pad 2: Net-(D43-Pad2) -> (no net)
- D44 pad 1: ROW3 -> (no net)
- D44 pad 2: Net-(D44-Pad2) -> (no net)
- D45 pad 1: ROW4 -> (no net)
- D45 pad 2: Net-(D45-Pad2) -> (no net)
- D46 pad 1: ROW0 -> (no net)
- D46 pad 2: Net-(D46-Pad2) -> (no net)
- D47 pad 1: ROW1 -> (no net)
- D47 pad 2: Net-(D47-Pad2) -> (no net)
- D48 pad 1: ROW2 -> (no net)
- D48 pad 2: Net-(D48-Pad2) -> (no net)
- D49 pad 1: ROW3 -> (no net)
- D49 pad 2: Net-(D49-Pad2) -> (no net)
- D5 pad 1: ROW4 -> (no net)
- D5 pad 2: Net-(D5-Pad2) -> (no net)
- D50 pad 1: ROW4 -> (no net)
- D50 pad 2: Net-(D50-Pad2) -> (no net)
- D51 pad 1: ROW0 -> (no net)
- D51 pad 2: Net-(D51-Pad2) -> (no net)
- D52 pad 1: ROW1 -> (no net)
- D52 pad 2: Net-(D52-Pad2) -> (no net)
- D53 pad 1: ROW2 -> (no net)
- D53 pad 2: Net-(D53-Pad2) -> (no net)
- D54 pad 1: ROW3 -> (no net)
- D54 pad 2: Net-(D54-Pad2) -> (no net)
- D55 pad 1: ROW4 -> (no net)
- D55 pad 2: Net-(D55-Pad2) -> (no net)
- D56 pad 1: ROW0 -> (no net)
- D56 pad 2: Net-(D56-Pad2) -> (no net)
- D57 pad 1: ROW1 -> (no net)
- D57 pad 2: Net-(D57-Pad2) -> (no net)
- D58 pad 1: ROW2 -> (no net)
- D58 pad 2: Net-(D58-Pad2) -> (no net)
- D59 pad 1: ROW3 -> (no net)
- D59 pad 2: Net-(D59-Pad2) -> (no net)
- D6 pad 1: ROW0 -> (no net)
- D6 pad 2: Net-(D6-Pad2) -> (no net)
- D60 pad 1: ROW4 -> (no net)
- D60 pad 2: Net-(D60-Pad2) -> (no net)
- D7 pad 1: ROW1 -> (no net)
- D7 pad 2: Net-(D7-Pad2) -> (no net)
- D8 pad 1: ROW2 -> (no net)
- D8 pad 2: Net-(D8-Pad2) -> (no net)
- D9 pad 1: ROW3 -> (no net)
- D9 pad 2: Net-(D9-Pad2) -> (no net)
- K1 pad 1: COL0 -> (no net)
- K1 pad 2: Net-(D1-Pad2) -> (no net)
- K10 pad 1: COL1 -> (no net)
- K10 pad 2: Net-(D10-Pad2) -> (no net)
- K11 pad 1: COL2 -> (no net)
- K11 pad 2: Net-(D11-Pad2) -> (no net)
- K12 pad 1: COL2 -> (no net)
- K12 pad 2: Net-(D12-Pad2) -> (no net)
- K13 pad 1: COL2 -> (no net)
- K13 pad 2: Net-(D13-Pad2) -> (no net)
- K14 pad 1: COL2 -> (no net)
- K14 pad 2: Net-(D14-Pad2) -> (no net)
- K15 pad 1: COL2 -> (no net)
- K15 pad 2: Net-(D15-Pad2) -> (no net)
- K16 pad 1: COL3 -> (no net)
- K16 pad 2: Net-(D16-Pad2) -> (no net)
- K17 pad 1: COL3 -> (no net)
- K17 pad 2: Net-(D17-Pad2) -> (no net)
- K18 pad 1: COL3 -> (no net)
- K18 pad 2: Net-(D18-Pad2) -> (no net)
- K19 pad 1: COL3 -> (no net)
- K19 pad 2: Net-(D19-Pad2) -> (no net)
- K2 pad 1: COL0 -> (no net)
- K2 pad 2: Net-(D2-Pad2) -> (no net)
- K20 pad 1: COL3 -> (no net)
- K20 pad 2: Net-(D20-Pad2) -> (no net)
- K21 pad 1: COL4 -> (no net)
- K21 pad 2: Net-(D21-Pad2) -> (no net)
- K22 pad 1: COL4 -> (no net)
- K22 pad 2: Net-(D22-Pad2) -> (no net)
- K23 pad 1: COL4 -> (no net)
- K23 pad 2: Net-(D23-Pad2) -> (no net)
- K24 pad 1: COL4 -> (no net)
- K24 pad 2: Net-(D24-Pad2) -> (no net)
- K25 pad 1: COL4 -> (no net)
- K25 pad 2: Net-(D25-Pad2) -> (no net)
- K26 pad 1: COL5 -> (no net)
- K26 pad 2: Net-(D26-Pad2) -> (no net)
- K27 pad 1: COL5 -> (no net)
- K27 pad 2: Net-(D27-Pad2) -> (no net)
- K28 pad 1: COL5 -> (no net)
- K28 pad 2: Net-(D28-Pad2) -> (no net)
- K29 pad 1: COL5 -> (no net)
- K29 pad 2: Net-(D29-Pad2) -> (no net)
- K3 pad 1: COL0 -> (no net)
- K3 pad 2: Net-(D3-Pad2) -> (no net)
- K30 pad 1: COL5 -> (no net)
- K30 pad 2: Net-(D30-Pad2) -> (no net)
- K31 pad 1: COL6 -> (no net)
- K31 pad 2: Net-(D31-Pad2) -> (no net)
- K32 pad 1: COL6 -> (no net)
- K32 pad 2: Net-(D32-Pad2) -> (no net)
- K33 pad 1: COL6 -> (no net)
- K33 pad 2: Net-(D33-Pad2) -> (no net)
- K34 pad 1: COL6 -> (no net)
- K34 pad 2: Net-(D34-Pad2) -> (no net)
- K35 pad 1: COL6 -> (no net)
- K35 pad 2: Net-(D35-Pad2) -> (no net)
- K36 pad 1: COL7 -> (no net)
- K36 pad 2: Net-(D36-Pad2) -> (no net)
- K37 pad 1: COL7 -> (no net)
- K37 pad 2: Net-(D37-Pad2) -> (no net)
- K38 pad 1: COL7 -> (no net)
- K38 pad 2: Net-(D38-Pad2) -> (no net)
- K39 pad 1: COL7 -> (no net)
- K39 pad 2: Net-(D39-Pad2) -> (no net)
- K4 pad 1: COL0 -> (no net)
- K4 pad 2: Net-(D4-Pad2) -> (no net)
- K40 pad 1: COL7 -> (no net)
- K40 pad 2: Net-(D40-Pad2) -> (no net)
- K41 pad 1: COL8 -> (no net)
- K41 pad 2: Net-(D41-Pad2) -> (no net)
- K42 pad 1: COL8 -> (no net)
- K42 pad 2: Net-(D42-Pad2) -> (no net)
- K43 pad 1: COL8 -> (no net)
- K43 pad 2: Net-(D43-Pad2) -> (no net)
- K44 pad 1: COL8 -> (no net)
- K44 pad 2: Net-(D44-Pad2) -> (no net)
- K45 pad 1: COL8 -> (no net)
- K45 pad 2: Net-(D45-Pad2) -> (no net)
- K46 pad 1: COL9 -> (no net)
- K46 pad 2: Net-(D46-Pad2) -> (no net)
- K47 pad 1: COL9 -> (no net)
- K47 pad 2: Net-(D47-Pad2) -> (no net)
- K48 pad 1: COL9 -> (no net)
- K48 pad 2: Net-(D48-Pad2) -> (no net)
- K49 pad 1: COL9 -> (no net)
- K49 pad 2: Net-(D49-Pad2) -> (no net)
- K5 pad 1: COL0 -> (no net)
- K5 pad 2: Net-(D5-Pad2) -> (no net)
- K50 pad 1: COL9 -> (no net)
- K50 pad 2: Net-(D50-Pad2) -> (no net)
- K51 pad 1: COL10 -> (no net)
- K51 pad 2: Net-(D51-Pad2) -> (no net)
- K52 pad 1: COL10 -> (no net)
- K52 pad 2: Net-(D52-Pad2) -> (no net)
- K53 pad 1: COL10 -> (no net)
- K53 pad 2: Net-(D53-Pad2) -> (no net)
- K54 pad 1: COL10 -> (no net)
- K54 pad 2: Net-(D54-Pad2) -> (no net)
- K55 pad 1: COL10 -> (no net)
- K55 pad 2: Net-(D55-Pad2) -> (no net)
- K56 pad 1: COL11 -> (no net)
- K56 pad 2: Net-(D56-Pad2) -> (no net)
- K57 pad 1: COL11 -> (no net)
- K57 pad 2: Net-(D57-Pad2) -> (no net)
- K58 pad 1: COL11 -> (no net)
- K58 pad 2: Net-(D58-Pad2) -> (no net)
- K59 pad 1: COL11 -> (no net)
- K59 pad 2: Net-(D59-Pad2) -> (no net)
- K6 pad 1: COL1 -> (no net)
- K6 pad 2: Net-(D6-Pad2) -> (no net)
- K60 pad 1: COL11 -> (no net)
- K60 pad 2: Net-(D60-Pad2) -> (no net)
- K7 pad 1: COL1 -> (no net)
- K7 pad 2: Net-(D7-Pad2) -> (no net)
- K8 pad 1: COL1 -> (no net)
- K8 pad 2: Net-(D8-Pad2) -> (no net)
- K9 pad 1: COL1 -> (no net)
- K9 pad 2: Net-(D9-Pad2) -> (no net)
- U1 pad 1: Net-(U1-Pad1) -> (no net)
- U1 pad 10: COL3 -> (no net)
- U1 pad 11: COL4 -> (no net)
- U1 pad 12: ROW4 -> (no net)
- U1 pad 13: ROW2 -> (no net)
- U1 pad 14: ROW3 -> (no net)
- U1 pad 15: Net-(U1-Pad15) -> (no net)
- U1 pad 16: GND -> (no net)
- U1 pad 17: Net-(U1-Pad17) -> (no net)
- U1 pad 18: Net-(U1-Pad18) -> (no net)
- U1 pad 19: Net-(U1-Pad19) -> (no net)
- U1 pad 2: Net-(U1-Pad2) -> (no net)
- U1 pad 20: Net-(U1-Pad20) -> (no net)
- U1 pad 21: Net-(U1-Pad21) -> (no net)
- U1 pad 22: Net-(U1-Pad22) -> (no net)
- U1 pad 23: Net-(U1-Pad23) -> (no net)
- U1 pad 24: Net-(U1-Pad24) -> (no net)
- U1 pad 25: COL7 -> (no net)
- U1 pad 26: COL1 -> (no net)
- U1 pad 27: COL8 -> (no net)
- U1 pad 28: Net-(U1-Pad28) -> (no net)
- U1 pad 29: Net-(U1-Pad29) -> (no net)
- U1 pad 3: Net-(U1-Pad3) -> (no net)
- U1 pad 30: COL9 -> (no net)
- U1 pad 31: COL10 -> (no net)
- U1 pad 32: ROW1 -> (no net)
- U1 pad 33: COL11 -> (no net)
- U1 pad 34: Net-(U1-Pad34) -> (no net)
- U1 pad 35: ROW0 -> (no net)
- U1 pad 36: COL0 -> (no net)
- U1 pad 4: Net-(U1-Pad4) -> (no net)
- U1 pad 5: COL5 -> (no net)
- U1 pad 6: COL6 -> (no net)
- U1 pad 7: Net-(U1-Pad7) -> (no net)
- U1 pad 8: Net-(U1-Pad8) -> (no net)
- U1 pad 9: COL2 -> (no net)
Routing:
- net (no net): track 0.00 -> 4697.3 mm, vias 41 -> 85
- net ROW3: track 382.3 -> 0.00 mm
- net ROW0: track 375.2 -> 0.00 mm
- net COL11: track 343.1 -> 0.00 mm
- net COL10: track 335.0 -> 0.00 mm, vias 1 -> 0
- net COL9: track 323.9 -> 0.00 mm, vias 1 -> 0
- net ROW2: track 284.0 -> 0.00 mm, vias 5 -> 0
- net ROW1: track 280.9 -> 0.00 mm, vias 4 -> 0
- net ROW4: track 277.9 -> 0.00 mm
- net COL8: track 275.3 -> 0.00 mm, vias 1 -> 0
- net COL7: track 270.9 -> 0.00 mm, vias 1 -> 0
- net COL6: track 216.2 -> 0.00 mm, vias 2 -> 0
- net COL5: track 198.1 -> 0.00 mm, vias 2 -> 0
- net COL0: track 187.4 -> 0.00 mm, vias 1 -> 0
- net COL3: track 183.1 -> 0.00 mm, vias 1 -> 0
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- added copper zone on B.Cu, net (none)
- added copper zone on F.Cu, net (none)
- removed copper zone on B.Cu, net GND
- removed copper zone on F.Cu, net GND
Other:
- board size 259.6 x 290.5 mm -> 259.6 x 289.8 mm

Commit message: Adding LEDs.
Parts:
- removed the G*** at (166.7, 302.4)
- removed the G*** at (281.0, 302.4)
- removed mouse-bite-2mm-slot (x6): VAL**, Panelization:mouse-bite-2mm-slot
- added L1: LED_sk2812_SM, SofleRGB:SK6812MINI_and_cherry, F.Cu at (119.1, 163.9)
- added L10: LED_sk2812_SM, SofleRGB:SK6812MINI_and_cherry, F.Cu at (138.1, 240.1)
- added L11: LED_sk2812_SM, SofleRGB:SK6812MINI_and_cherry, F.Cu at (157.2, 163.9)
- added L12: LED_sk2812_SM, SofleRGB:SK6812MINI_and_cherry, F.Cu at (157.2, 183.0)
- added L13: LED_sk2812_SM, SofleRGB:SK6812MINI_and_cherry, F.Cu at (157.2, 202.0)
- added L14: LED_sk2812_SM, SofleRGB:SK6812MINI_and_cherry, F.Cu at (157.2, 221.1)
- added L15: LED_sk2812_SM, SofleRGB:SK6812MINI_and_cherry, F.Cu at (157.2, 240.1)
- added L16: LED_sk2812_SM, SofleRGB:SK6812MINI_and_cherry, F.Cu at (176.2, 163.9)
- added L17: LED_sk2812_SM, SofleRGB:SK6812MINI_and_cherry, F.Cu at (176.2, 183.0)
- added L18: LED_sk2812_SM, SofleRGB:SK6812MINI_and_cherry, F.Cu at (176.2, 202.0)
- added L19: LED_sk2812_SM, SofleRGB:SK6812MINI_and_cherry, F.Cu at (176.2, 221.1)
- added L2: LED_sk2812_SM, SofleRGB:SK6812MINI_and_cherry, F.Cu at (119.1, 183.0)
- added L20: LED_sk2812_SM, SofleRGB:SK6812MINI_and_cherry, F.Cu at (176.2, 240.1)
- added L21: LED_sk2812_SM, SofleRGB:SK6812MINI_and_cherry, F.Cu at (195.3, 163.9)
- added L22: LED_sk2812_SM, SofleRGB:SK6812MINI_and_cherry, F.Cu at (195.3, 183.0)
- added L23: LED_sk2812_SM, SofleRGB:SK6812MINI_and_cherry, F.Cu at (195.3, 202.0)
- added L24: LED_sk2812_SM, SofleRGB:SK6812MINI_and_cherry, F.Cu at (195.3, 221.1)
- added L25: LED_sk2812_SM, SofleRGB:SK6812MINI_and_cherry, F.Cu at (195.3, 240.1)
- added L26: LED_sk2812_SM, SofleRGB:SK6812MINI_and_cherry, F.Cu at (214.3, 163.9)
- added L27: LED_sk2812_SM, SofleRGB:SK6812MINI_and_cherry, F.Cu at (214.3, 183.0)
- added L28: LED_sk2812_SM, SofleRGB:SK6812MINI_and_cherry, F.Cu at (214.3, 202.0)
- added L29: LED_sk2812_SM, SofleRGB:SK6812MINI_and_cherry, F.Cu at (214.3, 221.1)
- added L3: LED_sk2812_SM, SofleRGB:SK6812MINI_and_cherry, F.Cu at (119.1, 202.0)
- added L30: LED_sk2812_SM, SofleRGB:SK6812MINI_and_cherry, F.Cu at (214.3, 240.1)
- added L31: LED_sk2812_SM, SofleRGB:SK6812MINI_and_cherry, F.Cu at (233.4, 163.9)
- added L32: LED_sk2812_SM, SofleRGB:SK6812MINI_and_cherry, F.Cu at (233.4, 183.0)
- added L33: LED_sk2812_SM, SofleRGB:SK6812MINI_and_cherry, F.Cu at (233.4, 202.0)
- added L34: LED_sk2812_SM, SofleRGB:SK6812MINI_and_cherry, F.Cu at (233.4, 221.1)
- added L35: LED_sk2812_SM, SofleRGB:SK6812MINI_and_cherry, F.Cu at (233.4, 240.1)
- added L36: LED_sk2812_SM, SofleRGB:SK6812MINI_and_cherry, F.Cu at (252.4, 163.9)
- added L37: LED_sk2812_SM, SofleRGB:SK6812MINI_and_cherry, F.Cu at (252.4, 183.0)
- added L38: LED_sk2812_SM, SofleRGB:SK6812MINI_and_cherry, F.Cu at (252.4, 202.0)
- added L39: LED_sk2812_SM, SofleRGB:SK6812MINI_and_cherry, F.Cu at (252.4, 221.1)
- added L4: LED_sk2812_SM, SofleRGB:SK6812MINI_and_cherry, F.Cu at (119.1, 221.1)
- added L40: LED_sk2812_SM, SofleRGB:SK6812MINI_and_cherry, F.Cu at (252.4, 240.1)
- added L41: LED_sk2812_SM, SofleRGB:SK6812MINI_and_cherry, F.Cu at (271.5, 163.9)
- added L42: LED_sk2812_SM, SofleRGB:SK6812MINI_and_cherry, F.Cu at (271.5, 183.0)
- added L43: LED_sk2812_SM, SofleRGB:SK6812MINI_and_cherry, F.Cu at (271.5, 202.0)
- added L44: LED_sk2812_SM, SofleRGB:SK6812MINI_and_cherry, F.Cu at (271.5, 221.1)
- added L45: LED_sk2812_SM, SofleRGB:SK6812MINI_and_cherry, F.Cu at (271.5, 240.1)
- added L46: LED_sk2812_SM, SofleRGB:SK6812MINI_and_cherry, F.Cu at (290.5, 163.9)
- added L47: LED_sk2812_SM, SofleRGB:SK6812MINI_and_cherry, F.Cu at (290.5, 183.0)
- added L48: LED_sk2812_SM, SofleRGB:SK6812MINI_and_cherry, F.Cu at (290.5, 202.0)
- added L49: LED_sk2812_SM, SofleRGB:SK6812MINI_and_cherry, F.Cu at (290.5, 221.1)
- added L5: LED_sk2812_SM, SofleRGB:SK6812MINI_and_cherry, F.Cu at (119.1, 240.1)
- added L50: LED_sk2812_SM, SofleRGB:SK6812MINI_and_cherry, F.Cu at (290.5, 240.1)
- added L51: LED_sk2812_SM, SofleRGB:SK6812MINI_and_cherry, F.Cu at (309.6, 163.9)
- added L52: LED_sk2812_SM, SofleRGB:SK6812MINI_and_cherry, F.Cu at (309.6, 183.0)
- added L53: LED_sk2812_SM, SofleRGB:SK6812MINI_and_cherry, F.Cu at (309.6, 202.0)
- added L54: LED_sk2812_SM, SofleRGB:SK6812MINI_and_cherry, F.Cu at (309.6, 221.1)
- added L55: LED_sk2812_SM, SofleRGB:SK6812MINI_and_cherry, F.Cu at (309.6, 240.1)
- added L56: LED_sk2812_SM, SofleRGB:SK6812MINI_and_cherry, F.Cu at (328.6, 163.9)
- added L57: LED_sk2812_SM, SofleRGB:SK6812MINI_and_cherry, F.Cu at (328.6, 183.0)
- added L58: LED_sk2812_SM, SofleRGB:SK6812MINI_and_cherry, F.Cu at (328.6, 202.0)
- added L59: LED_sk2812_SM, SofleRGB:SK6812MINI_and_cherry, F.Cu at (328.6, 221.1)
- added L6: LED_sk2812_SM, SofleRGB:SK6812MINI_and_cherry, F.Cu at (138.1, 163.9)
- added L60: LED_sk2812_SM, SofleRGB:SK6812MINI_and_cherry, F.Cu at (328.6, 240.1)
- added L7: LED_sk2812_SM, SofleRGB:SK6812MINI_and_cherry, F.Cu at (138.1, 183.4)
- added L8: LED_sk2812_SM, SofleRGB:SK6812MINI_and_cherry, F.Cu at (138.1, 202.0)
- added L9: LED_sk2812_SM, SofleRGB:SK6812MINI_and_cherry, F.Cu at (138.1, 221.1)
- added T1: HOLE, SofleRGB:HOLE_M2_TH, F.Cu at (300.0, 173.4)
- added T10: HOLE, SofleRGB:HOLE_M2_TH, F.Cu at (204.8, 211.6)
- added T11: HOLE, SofleRGB:HOLE_M2_TH, F.Cu at (185.7, 230.6)
- added T12: HOLE, SofleRGB:HOLE_M2_TH, F.Cu at (147.6, 230.6)
- added T13: HOLE, SofleRGB:HOLE_M2_TH, F.Cu at (128.6, 211.6)
- added T14: HOLE, SofleRGB:HOLE_M2_TH, F.Cu at (128.6, 192.5)
- added T15: HOLE, SofleRGB:HOLE_M2_TH, F.Cu at (147.6, 173.4)
- added T16: HOLE, SofleRGB:HOLE_M2_TH, F.Cu at (185.7, 173.4)
- added T2: HOLE, SofleRGB:HOLE_M2_TH, F.Cu at (319.1, 192.5)
- added T3: HOLE, SofleRGB:HOLE_M2_TH, F.Cu at (319.1, 211.6)
- added T4: HOLE, SofleRGB:HOLE_M2_TH, F.Cu at (300.0, 230.6)
- added T5: HOLE, SofleRGB:HOLE_M2_TH, F.Cu at (261.9, 230.6)
- added T6: HOLE, SofleRGB:HOLE_M2_TH, F.Cu at (242.9, 211.6)
- added T7: HOLE, SofleRGB:HOLE_M2_TH, F.Cu at (242.9, 192.5)
- added T8: HOLE, SofleRGB:HOLE_M2_TH, F.Cu at (261.9, 173.4)
- added T9: HOLE, SofleRGB:HOLE_M2_TH, F.Cu at (204.8, 192.5)
- added TH1-1: HOLE, SofleRGB:M2_HOLE_PCB, F.Cu at (319.1, 76.2)
- added TH1-10: HOLE, SofleRGB:M2_HOLE_PCB, F.Cu at (185.7, 133.3)
- added TH1-11: HOLE, SofleRGB:M2_HOLE_PCB, F.Cu at (147.6, 133.3)
- added TH1-12: HOLE, SofleRGB:M2_HOLE_PCB, F.Cu at (128.6, 133.3)
- added TH1-13: HOLE, SofleRGB:M2_HOLE_PCB, F.Cu at (128.6, 114.3)
- added TH1-14: HOLE, SofleRGB:M2_HOLE_PCB, F.Cu at (128.6, 95.2)
- added TH1-15: HOLE, SofleRGB:M2_HOLE_PCB, F.Cu at (128.6, 76.2)
- added TH1-16: HOLE, SofleRGB:M2_HOLE_PCB, F.Cu at (147.6, 76.2)
- added TH1-17: HOLE, SofleRGB:M2_HOLE_PCB, F.Cu at (185.7, 76.2)
- added TH1-18: HOLE, SofleRGB:M2_HOLE_PCB, F.Cu at (204.8, 95.2)
- added TH1-19: HOLE, SofleRGB:M2_HOLE_PCB, F.Cu at (223.8, 76.2)
- added TH1-2: HOLE, SofleRGB:M2_HOLE_PCB, F.Cu at (319.1, 95.2)
- added TH1-20: HOLE, SofleRGB:M2_HOLE_PCB, F.Cu at (242.9, 95.2)
- added TH1-21: HOLE, SofleRGB:M2_HOLE_PCB, F.Cu at (261.9, 76.2)
- added TH1-22: HOLE, SofleRGB:M2_HOLE_PCB, F.Cu at (104.8, 133.3)
- added TH1-22: HOLE, SofleRGB:M2_HOLE_PCB, F.Cu at (83.3, 133.3)
- added TH1-22: HOLE, SofleRGB:M2_HOLE_PCB, F.Cu at (300.0, 76.2)
- added TH1-3: HOLE, SofleRGB:M2_HOLE_PCB, F.Cu at (319.1, 114.3)
- added TH1-4: HOLE, SofleRGB:M2_HOLE_PCB, F.Cu at (319.1, 133.3)
- added TH1-5: HOLE, SofleRGB:M2_HOLE_PCB, F.Cu at (300.0, 133.3)
- added TH1-6: HOLE, SofleRGB:M2_HOLE_PCB, F.Cu at (261.9, 133.3)
- added TH1-7: HOLE, SofleRGB:M2_HOLE_PCB, F.Cu at (242.9, 114.3)
- added TH1-8: HOLE, SofleRGB:M2_HOLE_PCB, F.Cu at (223.8, 133.3)
- added TH1-9: HOLE, SofleRGB:M2_HOLE_PCB, F.Cu at (204.8, 114.3)
- added TH2-1: HOLE, SofleRGB:M2_HOLE_PCB, F.Cu at (319.1, 173.4)
- added TH2-2: HOLE, SofleRGB:M2_HOLE_PCB, F.Cu at (319.1, 230.6)
- added TH2-3: HOLE, SofleRGB:M2_HOLE_PCB, F.Cu at (223.8, 230.6)
- added TH2-4: HOLE, SofleRGB:M2_HOLE_PCB, F.Cu at (128.6, 230.6)
- added TH2-5: HOLE, SofleRGB:M2_HOLE_PCB, F.Cu at (128.6, 173.4)
- added TH2-6: HOLE, SofleRGB:M2_HOLE_PCB, F.Cu at (223.8, 173.4)
- added TH3-1: HOLE, SofleRGB:M2_HOLE_PCB, F.Cu at (300.0, 270.7)
- added TH3-10: HOLE, SofleRGB:M2_HOLE_PCB, F.Cu at (204.8, 289.8)
- added TH3-11: HOLE, SofleRGB:M2_HOLE_PCB, F.Cu at (204.8, 308.8)
- added TH3-12: HOLE, SofleRGB:M2_HOLE_PCB, F.Cu at (185.7, 327.9)
- added TH3-13: HOLE, SofleRGB:M2_HOLE_PCB, F.Cu at (147.6, 327.9)
- added TH3-14: HOLE, SofleRGB:M2_HOLE_PCB, F.Cu at (128.6, 308.8)
- added TH3-15: HOLE, SofleRGB:M2_HOLE_PCB, F.Cu at (128.6, 289.8)
- added TH3-16: HOLE, SofleRGB:M2_HOLE_PCB, F.Cu at (147.6, 270.7)
- added TH3-2: HOLE, SofleRGB:M2_HOLE_PCB, F.Cu at (319.1, 289.8)
- added TH3-3: HOLE, SofleRGB:M2_HOLE_PCB, F.Cu at (319.1, 308.8)
- added TH3-4: HOLE, SofleRGB:M2_HOLE_PCB, F.Cu at (300.0, 327.9)
- added TH3-5: HOLE, SofleRGB:M2_HOLE_PCB, F.Cu at (261.9, 327.9)
- added TH3-6: HOLE, SofleRGB:M2_HOLE_PCB, F.Cu at (242.9, 308.8)
- added TH3-7: HOLE, SofleRGB:M2_HOLE_PCB, F.Cu at (242.9, 289.8)
- added TH3-8: HOLE, SofleRGB:M2_HOLE_PCB, F.Cu at (261.9, 270.7)
- added TH3-9: HOLE, SofleRGB:M2_HOLE_PCB, F.Cu at (185.7, 270.7)
- added U2: 0.91_oled_128x32, footprints:0.91_oled_128x32, F.Cu at (93.0, 202.1)
- added mouse-bite-2mm-slot-1: VAL1, Panelization:mouse-bite-2mm-slot, F.Cu at (147.1, 250.7)
- added mouse-bite-2mm-slot-2: VAL2, Panelization:mouse-bite-2mm-slot, F.Cu at (224.1, 250.7)
- added mouse-bite-2mm-slot-3: VAL3, Panelization:mouse-bite-2mm-slot, F.Cu at (300.1, 250.7)
- added mouse-bite-2mm-slot-4: VAL4, Panelization:mouse-bite-2mm-slot, F.Cu at (147.1, 153.4)
- added mouse-bite-2mm-slot-5: VAL5, Panelization:mouse-bite-2mm-slot, F.Cu at (224.1, 153.4)
- added mouse-bite-2mm-slot-6: VAL6, Panelization:mouse-bite-2mm-slot, F.Cu at (300.1, 153.4)
- D1, D10, D11, D12, D13, D14, D15, D16, D17, D18, D19, D2, D20, D21, D22, D23, D24, D25, D26, D27, D28, D29, D3, D30, D31, D32, D33, D34, D35, D36, D37, D38, D39, D4, D40, D41, D42, D43, D44, D45, D46, D47, D48, D49, D5, D50, D51, D52, D53, D54, D55, D56, D57, D58, D59, D6, D60, D7, D8, D9: footprint keyboard_parts:D_SOD123 -> keyboard_parts:D_SOD123_hand
- U1: moved to B.Cu
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Connections:
- D1 pad 1: (no net) -> ROW0
- D1 pad 2: (no net) -> Net-(D1-Pad2)
- D10 pad 1: (no net) -> ROW4
- D10 pad 2: (no net) -> Net-(D10-Pad2)
- D11 pad 1: (no net) -> ROW0
- D11 pad 2: (no net) -> Net-(D11-Pad2)
- D12 pad 1: (no net) -> ROW1
- D12 pad 2: (no net) -> Net-(D12-Pad2)
- D13 pad 1: (no net) -> ROW2
- D13 pad 2: (no net) -> Net-(D13-Pad2)
- D14 pad 1: (no net) -> ROW3
- D14 pad 2: (no net) -> Net-(D14-Pad2)
- D15 pad 1: (no net) -> ROW4
- D15 pad 2: (no net) -> Net-(D15-Pad2)
- D16 pad 1: (no net) -> ROW0
- D16 pad 2: (no net) -> Net-(D16-Pad2)
- D17 pad 1: (no net) -> ROW1
- D17 pad 2: (no net) -> Net-(D17-Pad2)
- D18 pad 1: (no net) -> ROW2
- D18 pad 2: (no net) -> Net-(D18-Pad2)
- D19 pad 1: (no net) -> ROW3
- D19 pad 2: (no net) -> Net-(D19-Pad2)
- D2 pad 1: (no net) -> ROW1
- D2 pad 2: (no net) -> Net-(D2-Pad2)
- D20 pad 1: (no net) -> ROW4
- D20 pad 2: (no net) -> Net-(D20-Pad2)
- D21 pad 1: (no net) -> ROW0
- D21 pad 2: (no net) -> Net-(D21-Pad2)
- D22 pad 1: (no net) -> ROW1
- D22 pad 2: (no net) -> Net-(D22-Pad2)
- D23 pad 1: (no net) -> ROW2
- D23 pad 2: (no net) -> Net-(D23-Pad2)
- D24 pad 1: (no net) -> ROW3
- D24 pad 2: (no net) -> Net-(D24-Pad2)
- D25 pad 1: (no net) -> ROW4
- D25 pad 2: (no net) -> Net-(D25-Pad2)
- D26 pad 1: (no net) -> ROW0
- D26 pad 2: (no net) -> Net-(D26-Pad2)
- D27 pad 1: (no net) -> ROW1
- D27 pad 2: (no net) -> Net-(D27-Pad2)
- D28 pad 1: (no net) -> ROW2
- D28 pad 2: (no net) -> Net-(D28-Pad2)
- D29 pad 1: (no net) -> ROW3
- D29 pad 2: (no net) -> Net-(D29-Pad2)
- D3 pad 1: (no net) -> ROW2
- D3 pad 2: (no net) -> Net-(D3-Pad2)
- D30 pad 1: (no net) -> ROW4
- D30 pad 2: (no net) -> Net-(D30-Pad2)
- D31 pad 1: (no net) -> ROW0
- D31 pad 2: (no net) -> Net-(D31-Pad2)
- D32 pad 1: (no net) -> ROW1
- D32 pad 2: (no net) -> Net-(D32-Pad2)
- D33 pad 1: (no net) -> ROW2
- D33 pad 2: (no net) -> Net-(D33-Pad2)
- D34 pad 1: (no net) -> ROW3
- D34 pad 2: (no net) -> Net-(D34-Pad2)
- D35 pad 1: (no net) -> ROW4
- D35 pad 2: (no net) -> Net-(D35-Pad2)
- D36 pad 1: (no net) -> ROW0
- D36 pad 2: (no net) -> Net-(D36-Pad2)
- D37 pad 1: (no net) -> ROW1
- D37 pad 2: (no net) -> Net-(D37-Pad2)
- D38 pad 1: (no net) -> ROW2
- D38 pad 2: (no net) -> Net-(D38-Pad2)
- D39 pad 1: (no net) -> ROW3
- D39 pad 2: (no net) -> Net-(D39-Pad2)
- D4 pad 1: (no net) -> ROW3
- D4 pad 2: (no net) -> Net-(D4-Pad2)
- D40 pad 1: (no net) -> ROW4
- D40 pad 2: (no net) -> Net-(D40-Pad2)
- D41 pad 1: (no net) -> ROW0
- D41 pad 2: (no net) -> Net-(D41-Pad2)
- D42 pad 1: (no net) -> ROW1
- D42 pad 2: (no net) -> Net-(D42-Pad2)
- D43 pad 1: (no net) -> ROW2
- D43 pad 2: (no net) -> Net-(D43-Pad2)
- D44 pad 1: (no net) -> ROW3
- D44 pad 2: (no net) -> Net-(D44-Pad2)
- D45 pad 1: (no net) -> ROW4
- D45 pad 2: (no net) -> Net-(D45-Pad2)
- D46 pad 1: (no net) -> ROW0
- D46 pad 2: (no net) -> Net-(D46-Pad2)
- D47 pad 1: (no net) -> ROW1
- D47 pad 2: (no net) -> Net-(D47-Pad2)
- D48 pad 1: (no net) -> ROW2
- D48 pad 2: (no net) -> Net-(D48-Pad2)
- D49 pad 1: (no net) -> ROW3
- D49 pad 2: (no net) -> Net-(D49-Pad2)
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Routing:
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- removed copper zone on B.Cu, net (none)
- removed copper zone on F.Cu, net (none)
Other:
- outline, holes or cut-outs redrawn
- board text added: "Powered by MK32 github.com/Galzai/MK32"
- board text removed: "Powered by MK32 https://github.com/Galzai/MK32"

Commit message: v1.1
Parts:
- removed the G*** at (223.8, 271.5)
- removed the G*** at (223.8, 328.6)
- removed the TH1-22 at (104.8, 133.3)
- removed the TH1-22 at (83.3, 133.3)
- removed the TH1-22 at (300.0, 76.2)
- added G***: LOGO, testboard:logo, F.Cu at (223.8, 272.2)
- added G***: LOGO, testboard:logo, F.Cu at (223.8, 329.4)
- added TH1-22: HOLE, SofleRGB:M2_HOLE_PCB, F.Cu at (300.0, 76.6)
- added TH1-22: HOLE, SofleRGB:M2_HOLE_PCB, F.Cu at (104.8, 133.7)
- added TH1-22: HOLE, SofleRGB:M2_HOLE_PCB, F.Cu at (83.3, 133.7)
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Connections:
- D1 pad 1: ROW0 -> (no net)
- D1 pad 2: Net-(D1-Pad2) -> (no net)
- D10 pad 1: ROW4 -> (no net)
- D10 pad 2: Net-(D10-Pad2) -> (no net)
- D11 pad 1: ROW0 -> (no net)
- D11 pad 2: Net-(D11-Pad2) -> (no net)
- D12 pad 1: ROW1 -> (no net)
- D12 pad 2: Net-(D12-Pad2) -> (no net)
- D13 pad 1: ROW2 -> (no net)
- D13 pad 2: Net-(D13-Pad2) -> (no net)
- D14 pad 1: ROW3 -> (no net)
- D14 pad 2: Net-(D14-Pad2) -> (no net)
- D15 pad 1: ROW4 -> (no net)
- D15 pad 2: Net-(D15-Pad2) -> (no net)
- D16 pad 1: ROW0 -> (no net)
- D16 pad 2: Net-(D16-Pad2) -> (no net)
- D17 pad 1: ROW1 -> (no net)
- D17 pad 2: Net-(D17-Pad2) -> (no net)
- D18 pad 1: ROW2 -> (no net)
- D18 pad 2: Net-(D18-Pad2) -> (no net)
- D19 pad 1: ROW3 -> (no net)
- D19 pad 2: Net-(D19-Pad2) -> (no net)
- D2 pad 1: ROW1 -> (no net)
- D2 pad 2: Net-(D2-Pad2) -> (no net)
- D20 pad 1: ROW4 -> (no net)
- D20 pad 2: Net-(D20-Pad2) -> (no net)
- D21 pad 1: ROW0 -> (no net)
- D21 pad 2: Net-(D21-Pad2) -> (no net)
- D22 pad 1: ROW1 -> (no net)
- D22 pad 2: Net-(D22-Pad2) -> (no net)
- D23 pad 1: ROW2 -> (no net)
- D23 pad 2: Net-(D23-Pad2) -> (no net)
- D24 pad 1: ROW3 -> (no net)
- D24 pad 2: Net-(D24-Pad2) -> (no net)
- D25 pad 1: ROW4 -> (no net)
- D25 pad 2: Net-(D25-Pad2) -> (no net)
- D26 pad 1: ROW0 -> (no net)
- D26 pad 2: Net-(D26-Pad2) -> (no net)
- D27 pad 1: ROW1 -> (no net)
- D27 pad 2: Net-(D27-Pad2) -> (no net)
- D28 pad 1: ROW2 -> (no net)
- D28 pad 2: Net-(D28-Pad2) -> (no net)
- D29 pad 1: ROW3 -> (no net)
- D29 pad 2: Net-(D29-Pad2) -> (no net)
- D3 pad 1: ROW2 -> (no net)
- D3 pad 2: Net-(D3-Pad2) -> (no net)
- D30 pad 1: ROW4 -> (no net)
- D30 pad 2: Net-(D30-Pad2) -> (no net)
- D31 pad 1: ROW0 -> (no net)
- D31 pad 2: Net-(D31-Pad2) -> (no net)
- D32 pad 1: ROW1 -> (no net)
- D32 pad 2: Net-(D32-Pad2) -> (no net)
- D33 pad 1: ROW2 -> (no net)
- D33 pad 2: Net-(D33-Pad2) -> (no net)
- D34 pad 1: ROW3 -> (no net)
- D34 pad 2: Net-(D34-Pad2) -> (no net)
- D35 pad 1: ROW4 -> (no net)
- D35 pad 2: Net-(D35-Pad2) -> (no net)
- D36 pad 1: ROW0 -> (no net)
- D36 pad 2: Net-(D36-Pad2) -> (no net)
- D37 pad 1: ROW1 -> (no net)
- D37 pad 2: Net-(D37-Pad2) -> (no net)
- D38 pad 1: ROW2 -> (no net)
- D38 pad 2: Net-(D38-Pad2) -> (no net)
- D39 pad 1: ROW3 -> (no net)
- D39 pad 2: Net-(D39-Pad2) -> (no net)
- D4 pad 1: ROW3 -> (no net)
- D4 pad 2: Net-(D4-Pad2) -> (no net)
- D40 pad 1: ROW4 -> (no net)
- D40 pad 2: Net-(D40-Pad2) -> (no net)
- D41 pad 1: ROW0 -> (no net)
- D41 pad 2: Net-(D41-Pad2) -> (no net)
- D42 pad 1: ROW1 -> (no net)
- D42 pad 2: Net-(D42-Pad2) -> (no net)
- D43 pad 1: ROW2 -> (no net)
- D43 pad 2: Net-(D43-Pad2) -> (no net)
- D44 pad 1: ROW3 -> (no net)
- D44 pad 2: Net-(D44-Pad2) -> (no net)
- D45 pad 1: ROW4 -> (no net)
- D45 pad 2: Net-(D45-Pad2) -> (no net)
- D46 pad 1: ROW0 -> (no net)
- D46 pad 2: Net-(D46-Pad2) -> (no net)
- D47 pad 1: ROW1 -> (no net)
- D47 pad 2: Net-(D47-Pad2) -> (no net)
- D48 pad 1: ROW2 -> (no net)
- D48 pad 2: Net-(D48-Pad2) -> (no net)
- D49 pad 1: ROW3 -> (no net)
- D49 pad 2: Net-(D49-Pad2) -> (no net)
- D5 pad 1: ROW4 -> (no net)
- D5 pad 2: Net-(D5-Pad2) -> (no net)
- D50 pad 1: ROW4 -> (no net)
- D50 pad 2: Net-(D50-Pad2) -> (no net)
- D51 pad 1: ROW0 -> (no net)
- D51 pad 2: Net-(D51-Pad2) -> (no net)
- D52 pad 1: ROW1 -> (no net)
- D52 pad 2: Net-(D52-Pad2) -> (no net)
- D53 pad 1: ROW2 -> (no net)
- D53 pad 2: Net-(D53-Pad2) -> (no net)
- D54 pad 1: ROW3 -> (no net)
- D54 pad 2: Net-(D54-Pad2) -> (no net)
- D55 pad 1: ROW4 -> (no net)
- D55 pad 2: Net-(D55-Pad2) -> (no net)
- D56 pad 1: ROW0 -> (no net)
- D56 pad 2: Net-(D56-Pad2) -> (no net)
- D57 pad 1: ROW1 -> (no net)
- D57 pad 2: Net-(D57-Pad2) -> (no net)
- D58 pad 1: ROW2 -> (no net)
- D58 pad 2: Net-(D58-Pad2) -> (no net)
- D59 pad 1: ROW3 -> (no net)
- D59 pad 2: Net-(D59-Pad2) -> (no net)
- D6 pad 1: ROW0 -> (no net)
- D6 pad 2: Net-(D6-Pad2) -> (no net)
- D60 pad 1: ROW4 -> (no net)
- D60 pad 2: Net-(D60-Pad2) -> (no net)
- D7 pad 1: ROW1 -> (no net)
- D7 pad 2: Net-(D7-Pad2) -> (no net)
- D8 pad 1: ROW2 -> (no net)
- D8 pad 2: Net-(D8-Pad2) -> (no net)
- D9 pad 1: ROW3 -> (no net)
- D9 pad 2: Net-(D9-Pad2) -> (no net)
- K1 pad 1: COL0 -> (no net)
- K1 pad 2: Net-(D1-Pad2) -> (no net)
- K10 pad 1: COL1 -> (no net)
- K10 pad 2: Net-(D10-Pad2) -> (no net)
- K11 pad 1: COL2 -> (no net)
- K11 pad 2: Net-(D11-Pad2) -> (no net)
- K12 pad 1: COL2 -> (no net)
- K12 pad 2: Net-(D12-Pad2) -> (no net)
- K13 pad 1: COL2 -> (no net)
- K13 pad 2: Net-(D13-Pad2) -> (no net)
- K14 pad 1: COL2 -> (no net)
- K14 pad 2: Net-(D14-Pad2) -> (no net)
- K15 pad 1: COL2 -> (no net)
- K15 pad 2: Net-(D15-Pad2) -> (no net)
- K16 pad 1: COL3 -> (no net)
- K16 pad 2: Net-(D16-Pad2) -> (no net)
- K17 pad 1: COL3 -> (no net)
- K17 pad 2: Net-(D17-Pad2) -> (no net)
- K18 pad 1: COL3 -> (no net)
- K18 pad 2: Net-(D18-Pad2) -> (no net)
- K19 pad 1: COL3 -> (no net)
- K19 pad 2: Net-(D19-Pad2) -> (no net)
- K2 pad 1: COL0 -> (no net)
- K2 pad 2: Net-(D2-Pad2) -> (no net)
- K20 pad 1: COL3 -> (no net)
- K20 pad 2: Net-(D20-Pad2) -> (no net)
- K21 pad 1: COL4 -> (no net)
- K21 pad 2: Net-(D21-Pad2) -> (no net)
- K22 pad 1: COL4 -> (no net)
- K22 pad 2: Net-(D22-Pad2) -> (no net)
- K23 pad 1: COL4 -> (no net)
- K23 pad 2: Net-(D23-Pad2) -> (no net)
- K24 pad 1: COL4 -> (no net)
- K24 pad 2: Net-(D24-Pad2) -> (no net)
- K25 pad 1: COL4 -> (no net)
- K25 pad 2: Net-(D25-Pad2) -> (no net)
- K26 pad 1: COL5 -> (no net)
- K26 pad 2: Net-(D26-Pad2) -> (no net)
- K27 pad 1: COL5 -> (no net)
- K27 pad 2: Net-(D27-Pad2) -> (no net)
- K28 pad 1: COL5 -> (no net)
- K28 pad 2: Net-(D28-Pad2) -> (no net)
- K29 pad 1: COL5 -> (no net)
- K29 pad 2: Net-(D29-Pad2) -> (no net)
- K3 pad 1: COL0 -> (no net)
- K3 pad 2: Net-(D3-Pad2) -> (no net)
- K30 pad 1: COL5 -> (no net)
- K30 pad 2: Net-(D30-Pad2) -> (no net)
- K31 pad 1: COL6 -> (no net)
- K31 pad 2: Net-(D31-Pad2) -> (no net)
- K32 pad 1: COL6 -> (no net)
- K32 pad 2: Net-(D32-Pad2) -> (no net)
- K33 pad 1: COL6 -> (no net)
- K33 pad 2: Net-(D33-Pad2) -> (no net)
- K34 pad 1: COL6 -> (no net)
- K34 pad 2: Net-(D34-Pad2) -> (no net)
- K35 pad 1: COL6 -> (no net)
- K35 pad 2: Net-(D35-Pad2) -> (no net)
- K36 pad 1: COL7 -> (no net)
- K36 pad 2: Net-(D36-Pad2) -> (no net)
- K37 pad 1: COL7 -> (no net)
- K37 pad 2: Net-(D37-Pad2) -> (no net)
- K38 pad 1: COL7 -> (no net)
- K38 pad 2: Net-(D38-Pad2) -> (no net)
- K39 pad 1: COL7 -> (no net)
- K39 pad 2: Net-(D39-Pad2) -> (no net)
- K4 pad 1: COL0 -> (no net)
- K4 pad 2: Net-(D4-Pad2) -> (no net)
- K40 pad 1: COL7 -> (no net)
- K40 pad 2: Net-(D40-Pad2) -> (no net)
- K41 pad 1: COL8 -> (no net)
- K41 pad 2: Net-(D41-Pad2) -> (no net)
- K42 pad 1: COL8 -> (no net)
- K42 pad 2: Net-(D42-Pad2) -> (no net)
- K43 pad 1: COL8 -> (no net)
- K43 pad 2: Net-(D43-Pad2) -> (no net)
- K44 pad 1: COL8 -> (no net)
- K44 pad 2: Net-(D44-Pad2) -> (no net)
- K45 pad 1: COL8 -> (no net)
- K45 pad 2: Net-(D45-Pad2) -> (no net)
- K46 pad 1: COL9 -> (no net)
- K46 pad 2: Net-(D46-Pad2) -> (no net)
- K47 pad 1: COL9 -> (no net)
- K47 pad 2: Net-(D47-Pad2) -> (no net)
- K48 pad 1: COL9 -> (no net)
- K48 pad 2: Net-(D48-Pad2) -> (no net)
- K49 pad 1: COL9 -> (no net)
- K49 pad 2: Net-(D49-Pad2) -> (no net)
- K5 pad 1: COL0 -> (no net)
- K5 pad 2: Net-(D5-Pad2) -> (no net)
- K50 pad 1: COL9 -> (no net)
- K50 pad 2: Net-(D50-Pad2) -> (no net)
- K51 pad 1: COL10 -> (no net)
- K51 pad 2: Net-(D51-Pad2) -> (no net)
- K52 pad 1: COL10 -> (no net)
- K52 pad 2: Net-(D52-Pad2) -> (no net)
- K53 pad 1: COL10 -> (no net)
- K53 pad 2: Net-(D53-Pad2) -> (no net)
- K54 pad 1: COL10 -> (no net)
- K54 pad 2: Net-(D54-Pad2) -> (no net)
- K55 pad 1: COL10 -> (no net)
- K55 pad 2: Net-(D55-Pad2) -> (no net)
- K56 pad 1: COL11 -> (no net)
- K56 pad 2: Net-(D56-Pad2) -> (no net)
- K57 pad 1: COL11 -> (no net)
- K57 pad 2: Net-(D57-Pad2) -> (no net)
- K58 pad 1: COL11 -> (no net)
- K58 pad 2: Net-(D58-Pad2) -> (no net)
- K59 pad 1: COL11 -> (no net)
- K59 pad 2: Net-(D59-Pad2) -> (no net)
- K6 pad 1: COL1 -> (no net)
- K6 pad 2: Net-(D6-Pad2) -> (no net)
- K60 pad 1: COL11 -> (no net)
- K60 pad 2: Net-(D60-Pad2) -> (no net)
- K7 pad 1: COL1 -> (no net)
- K7 pad 2: Net-(D7-Pad2) -> (no net)
- K8 pad 1: COL1 -> (no net)
- K8 pad 2: Net-(D8-Pad2) -> (no net)
- K9 pad 1: COL1 -> (no net)
- K9 pad 2: Net-(D9-Pad2) -> (no net)
- L1 pad 1: Net-(L1-Pad1) -> (no net)
- L1 pad 2: GND -> (no net)
- L1 pad 3: LED -> (no net)
- L1 pad 4: VCC -> (no net)
- L10 pad 1: Net-(L10-Pad1) -> (no net)
- L10 pad 2: GND -> (no net)
- L10 pad 3: Net-(L10-Pad3) -> (no net)
- L10 pad 4: VCC -> (no net)
- L11 pad 1: Net-(L11-Pad1) -> (no net)
- L11 pad 2: GND -> (no net)
- L11 pad 3: Net-(L10-Pad1) -> (no net)
- L11 pad 4: VCC -> (no net)
- L12 pad 1: Net-(L12-Pad1) -> (no net)
- L12 pad 2: GND -> (no net)
- L12 pad 3: Net-(L11-Pad1) -> (no net)
- L12 pad 4: VCC -> (no net)
- L13 pad 1: Net-(L13-Pad1) -> (no net)
- L13 pad 2: GND -> (no net)
- L13 pad 3: Net-(L12-Pad1) -> (no net)
- L13 pad 4: VCC -> (no net)
- L14 pad 1: Net-(L14-Pad1) -> (no net)
- L14 pad 2: GND -> (no net)
- L14 pad 3: Net-(L13-Pad1) -> (no net)
- L14 pad 4: VCC -> (no net)
- L15 pad 1: Net-(L15-Pad1) -> (no net)
- L15 pad 2: GND -> (no net)
- L15 pad 3: Net-(L14-Pad1) -> (no net)
- L15 pad 4: VCC -> (no net)
- L16 pad 1: Net-(L16-Pad1) -> (no net)
- L16 pad 2: GND -> (no net)
- L16 pad 3: Net-(L15-Pad1) -> (no net)
- L16 pad 4: VCC -> (no net)
- L17 pad 1: Net-(L17-Pad1) -> (no net)
- L17 pad 2: GND -> (no net)
- L17 pad 3: Net-(L16-Pad1) -> (no net)
- L17 pad 4: VCC -> (no net)
- L18 pad 1: Net-(L18-Pad1) -> (no net)
- L18 pad 2: GND -> (no net)
- L18 pad 3: Net-(L17-Pad1) -> (no net)
- L18 pad 4: VCC -> (no net)
- L19 pad 1: Net-(L19-Pad1) -> (no net)
- L19 pad 2: GND -> (no net)
- L19 pad 3: Net-(L18-Pad1) -> (no net)
- L19 pad 4: VCC -> (no net)
- L2 pad 1: Net-(L2-Pad1) -> (no net)
- L2 pad 2: GND -> (no net)
- L2 pad 3: Net-(L1-Pad1) -> (no net)
- L2 pad 4: VCC -> (no net)
- L20 pad 1: Net-(L20-Pad1) -> (no net)
- L20 pad 2: GND -> (no net)
- L20 pad 3: Net-(L19-Pad1) -> (no net)
- L20 pad 4: VCC -> (no net)
- L21 pad 1: Net-(L21-Pad1) -> (no net)
- L21 pad 2: GND -> (no net)
- L21 pad 3: Net-(L20-Pad1) -> (no net)
- L21 pad 4: VCC -> (no net)
- L22 pad 1: Net-(L22-Pad1) -> (no net)
- L22 pad 2: GND -> (no net)
- L22 pad 3: Net-(L21-Pad1) -> (no net)
- L22 pad 4: VCC -> (no net)
- L23 pad 1: Net-(L23-Pad1) -> (no net)
- L23 pad 2: GND -> (no net)
- L23 pad 3: Net-(L22-Pad1) -> (no net)
- L23 pad 4: VCC -> (no net)
- L24 pad 1: Net-(L24-Pad1) -> (no net)
- L24 pad 2: GND -> (no net)
- L24 pad 3: Net-(L23-Pad1) -> (no net)
- L24 pad 4: VCC -> (no net)
- L25 pad 1: Net-(L25-Pad1) -> (no net)
- L25 pad 2: GND -> (no net)
- L25 pad 3: Net-(L24-Pad1) -> (no net)
- L25 pad 4: VCC -> (no net)
- L26 pad 1: Net-(L26-Pad1) -> (no net)
- L26 pad 2: GND -> (no net)
- L26 pad 3: Net-(L25-Pad1) -> (no net)
- L26 pad 4: VCC -> (no net)
- L27 pad 1: Net-(L27-Pad1) -> (no net)
- L27 pad 2: GND -> (no net)
- L27 pad 3: Net-(L26-Pad1) -> (no net)
- L27 pad 4: VCC -> (no net)
- L28 pad 1: Net-(L28-Pad1) -> (no net)
- L28 pad 2: GND -> (no net)
- L28 pad 3: Net-(L27-Pad1) -> (no net)
- L28 pad 4: VCC -> (no net)
- L29 pad 1: Net-(L29-Pad1) -> (no net)
- L29 pad 2: GND -> (no net)
- L29 pad 3: Net-(L28-Pad1) -> (no net)
- L29 pad 4: VCC -> (no net)
- L3 pad 1: Net-(L3-Pad1) -> (no net)
- L3 pad 2: GND -> (no net)
- L3 pad 3: Net-(L2-Pad1) -> (no net)
- L3 pad 4: VCC -> (no net)
- L30 pad 1: Net-(L30-Pad1) -> (no net)
- L30 pad 2: GND -> (no net)
- L30 pad 3: Net-(L29-Pad1) -> (no net)
- L30 pad 4: VCC -> (no net)
- L31 pad 1: Net-(L31-Pad1) -> (no net)
- L31 pad 2: GND -> (no net)
- L31 pad 3: Net-(L30-Pad1) -> (no net)
- L31 pad 4: VCC -> (no net)
- L32 pad 1: Net-(L32-Pad1) -> (no net)
- L32 pad 2: GND -> (no net)
- L32 pad 3: Net-(L31-Pad1) -> (no net)
- L32 pad 4: VCC -> (no net)
- L33 pad 1: Net-(L33-Pad1) -> (no net)
- L33 pad 2: GND -> (no net)
- L33 pad 3: Net-(L32-Pad1) -> (no net)
- L33 pad 4: VCC -> (no net)
- L34 pad 1: Net-(L34-Pad1) -> (no net)
- L34 pad 2: GND -> (no net)
- L34 pad 3: Net-(L33-Pad1) -> (no net)
- L34 pad 4: VCC -> (no net)
- L35 pad 1: Net-(L35-Pad1) -> (no net)
- L35 pad 2: GND -> (no net)
- L35 pad 3: Net-(L34-Pad1) -> (no net)
- L35 pad 4: VCC -> (no net)
- L36 pad 1: Net-(L36-Pad1) -> (no net)
- L36 pad 2: GND -> (no net)
- L36 pad 3: Net-(L35-Pad1) -> (no net)
- L36 pad 4: VCC -> (no net)
- L37 pad 1: Net-(L37-Pad1) -> (no net)
- L37 pad 2: GND -> (no net)
- L37 pad 3: Net-(L36-Pad1) -> (no net)
- L37 pad 4: VCC -> (no net)
- L38 pad 1: Net-(L38-Pad1) -> (no net)
- L38 pad 2: GND -> (no net)
- L38 pad 3: Net-(L37-Pad1) -> (no net)
- L38 pad 4: VCC -> (no net)
- L39 pad 1: Net-(L39-Pad1) -> (no net)
- L39 pad 2: GND -> (no net)
- L39 pad 3: Net-(L38-Pad1) -> (no net)
- L39 pad 4: VCC -> (no net)
- L4 pad 1: Net-(L4-Pad1) -> (no net)
- L4 pad 2: GND -> (no net)
- L4 pad 3: Net-(L3-Pad1) -> (no net)
- L4 pad 4: VCC -> (no net)
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Routing:
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